File: PowerBoard.kicad_sch (KiCad schematic)
At the start: 50 parts

Commit message: Update PowerBoard.kicad_sch
Parts:
- R11, R5: value 24.7k -> 24.9k
Changed lines of the file:
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@@
 			)
 		)
-		(property "Value" "24.7k"
+		(property "Value" "24.9k"
 			(at 156.21 74.9299 0)
 			(effects
@@
 			)
 		)
-		(property "Value" "24.7k"
+		(property "Value" "24.9k"
 			(at 19.05 64.7699 0)
 			(effects

Commit message: finished schematic
Parts:
- removed C14: 4.7uF, symbol Device:C
- added C29: 10uF, Capacitor_SMD:C_1206_3216Metric, symbol Device:C
- added D2: D_Zener, Package_TO_SOT_SMD:SOT-23, symbol Device:D_Zener
- added D3, D4, D5: LED_Purple, symbol Device:LED
- added Q1: SQJ409EP, Package_SO:PowerPAK_SO-8L_Single, symbol Transistor_FET:SQJ409EP
- added R15, R18: 20k, Resistor_SMD:R_0603_1608Metric, symbol Device:R
- added R16, R17: 90k, Resistor_SMD:R_0603_1608Metric, symbol Device:R
- added R19, R20, R8: 1k, Resistor_SMD:R_0603_1608Metric, symbol Device:R
- added R6: 100k, Resistor_SMD:R_0603_1608Metric, symbol Device:R
- added U8: (no value), symbol PowerBoard:PowerOutput
- added U9: (no value), symbol powerBoardSchool:4x1_Header_Male
- C1: value C -> 1uF; footprint (none) -> Capacitor_SMD:C_0603_1608Metric
- C10, C11, C12, C21, C23, C25, C26, C8: footprint (none) -> Capacitor_SMD:C_1210_3225Metric
- C13, C24, C27, C5: footprint (none) -> Capacitor_SMD:CP_Elec_8x10.5
- C15: value 22uF -> 10uF; footprint (none) -> Capacitor_SMD:C_1206_3216Metric
- C16, C18, C19, C20, C28, C3, C4, C6, C7, C9: footprint (none) -> Capacitor_SMD:C_0603_1608Metric
- C17, C22: value 4.7uF -> 10uF; footprint (none) -> Capacitor_SMD:C_1206_3216Metric
- C2: value C -> 22uF; footprint (none) -> Capacitor_SMD:C_1210_3225Metric
- D1: footprint (none) -> Diode_SMD:D_SMA
- R1, R10, R11, R12, R13, R14, R2, R3, R4, R5, R7, R9: footprint (none) -> Resistor_SMD:R_0603_1608Metric
- U1, U2, U3, U4, U5, U6, U7: value ~ -> (none)
Connections:
- net +3V3: now also U5.2 (VOUT), R20.1
- net +5V: now also U7.2 (VOUT), R19.1
- net +6V: now also U3.2 (VOUT), R8.1
- net +VBAT_PRO: now also C29.1, D2.1 (K), Q1.1 (S), Q1.2 (S), Q1.3 (S), R16.1, R17.1, U8.2 (VOUT); no longer U1.7 (EN/SYNC), U4.7 (EN/SYNC)
- net GND: now also U2.1 (GND), U3.1 (GND), U5.1 (GND), U7.1 (GND), C29.2, D3.1 (K), D4.1 (K), D5.1 (K), R15.2, R18.2, R6.2, U8.1 (GND), U9.3, U9.4
- net PGOOD_5V: now also U9.2
- net PGOOD_6V: now also U9.1
- net at U2.2 (VIN): now also Q1.5 (D)
- new net: D5.2 (A), R20.2
- new net: D2.2 (A), Q1.4 (G), R6.1
- new net: R15.1, R16.2, U1.7 (EN/SYNC)
- new net: D3.2 (A), R8.2
- new net: D4.2 (A), R19.2
- new net: R17.2, R18.1, U4.7 (EN/SYNC)
Other:
- note added: "+VPROT(7V-27V) -> 5V Buck (6A Max)"
- note added: "+VPROT(7V-27V) -> 6V Buck (6A Max)"
- note added: "5V -> 3.3V LDO(1A max)"
- note added: "PGOOD Header Male"
- note added: "Power Out + Power LEDs"
- note added: "VBAT -> VPROT(7V-27V)"
- moved on the sheet: C1, C10, C11, C12, C13, C15, C16, C17, C18, C19, C2, C20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

Commit message: started layout
Parts:
- removed U5: (no value), symbol PowerBoard:PowerOutput
- added U5: (no value), PowerBoard:LowCurrentPad, symbol PowerBoard:PowerOutputLow
- D3, D4, D5: footprint (none) -> LED_SMD:LED_0603_1608Metric
- L1, L2: footprint (none) -> PowerBoard:Inductor_11.5_10
- U2: footprint (none) -> PowerBoard:HighCurrentPad
- U3, U7, U8: footprint (none) -> PowerBoard:ScrewTerminal
- U9: footprint (none) -> PowerBoard:4x1_2.54mmPitch
Connections:
- net +3V3: now also U5.2 (VOUT)
- net GND: now also U6.9 (GND), U5.1 (GND)
- net at R11.2: now also U4.6 (RT); no longer U1.6 (RT)
- net at R2.1: now also U1.6 (RT); no longer U4.6 (RT)
Other:
- moved on the sheet: D5, R11, R2

Commit message: finsihed main routing
Parts:
- added U10, U11, U12, U13: (no value), powerBoardSchool:Unbenannt, symbol powerBoardSchool:M2_Screw
- D1: footprint Diode_SMD:D_SMA -> Package_TO_SOT_SMD:SOT-23-3
Connections:
- net GND: now also U10.1, U11.1, U12.1, U13.1
Other:
- title: PowerBoard -> Neutron PowerBoard
- moved on the sheet: U9

Commit message: increased hole size
Parts:
- R2: value 33k -> 33.2k
Changed lines of the file:
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@@
 			)
 		)
-		(property "Value" "33k"
+		(property "Value" "33.2k"
 			(at 41.91 69.8499 0)
 			(show_name no)

Commit message: added LCSC codes
Parts:
- C1, C16, C6: LCSC Part # (none) -> C59782
- C10, C11, C12, C2, C21, C23, C25, C26, C8: LCSC Part # (none) -> C55530
- C13, C27: LCSC Part # (none) -> C497589
- C15, C17, C22, C29: LCSC Part # (none) -> C89632
- C18, C19, C20, C3, C4, C7: LCSC Part # (none) -> C1591
- C24, C5: LCSC Part # (none) -> C278406
- C28, C9: LCSC Part # (none) -> C1653
- D1: LCSC Part # (none) -> C545546
- D2: LCSC Part # (none) -> C108437
- D3, D4, D5: LCSC Part # (none) -> C7496831
- L1, L2: LCSC Part # (none) -> C49140770
- Q1: LCSC Part # (none) -> C727776
- R1, R12, R4, R6, R9: LCSC Part # (none) -> C2906980
- R10, R7: LCSC Part # (none) -> C2906981
- R11, R5: LCSC Part # (none) -> C2930080
- R13, R15, R18: LCSC Part # (none) -> C2907011
- R14, R19, R20, R3, R8: LCSC Part # (none) -> C2907002
- R16, R17: LCSC Part # (none) -> C2907077
- R2: LCSC Part # (none) -> C2933200
- U1, U4: LCSC Part # (none) -> C2876600
- U3, U7, U8: footprint PowerBoard:ScrewTerminal -> PowerBoard:HighCurrentPad
- U6: LCSC Part # (none) -> C2873382
